File: SEPIC/SEPIC.kicad_sch (KiCad schematic)
At the start: 20 parts, among them J1 Screw Terminal, J2 Barrel Jack, J3 Pin Header, J4 Screw Terminal, Q1 IRF520N, U1 HCPL-3120

Commit message: Imagenes PCB
Parts:
- C4: value 22u -> 10u; footprint Capacitor_THT:C_Radial_D8.0mm_H11.5mm_P3.50mm -> Capacitor_THT:C_Radial_D6.3mm_H7.0mm_P2.50mm
- L1: value 3m -> 2m
Other:
- moved on the sheet: D1
Changed lines of the file:
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@@
+	)
+	(junction
+		(at 109.22 73.66)
+		(diameter 0)
+		(color 0 0 0 0)
+	)
+	(junction
+		(at 54.61 67.31)
+		(diameter 0)
+		(color 0 0 0 0)
+	)
+	(junction
+		(at 93.98 92.71)
+		(diameter 0)
+		(color 0 0 0 0)
+	)
+	(junction
+		(at 153.67 36.83)
+		(diameter 0)
+		(color 0 0 0 0)
 	)
 	(junction
@@
 	)
 	(junction
-		(at 109.22 73.66)
-		(diameter 0)
-		(color 0 0 0 0)
-	)
-	(junction
-		(at 54.61 67.31)
-		(diameter 0)
-		(color 0 0 0 0)
-	)
-	(junction
-		(at 93.98 92.71)
-		(diameter 0)
-		(color 0 0 0 0)
-	)
-	(junction
-		(at 153.67 36.83)
-		(diameter 0)
-		(color 0 0 0 0)
-	)
-	(junction
 		(at 109.22 86.36)
 		(diameter 0)
@@
 	(wire
 		(pts
-			(xy 93.98 67.31) (xy 97.79 67.31)
+			(xy 93.98 67.31) (xy 96.52 67.31)
 		)
 		(stroke
@@
 	(wire
 		(pts
-			(xy 105.41 67.31) (xy 109.22 67.31)
-		)
-		(stroke
-			(width 0)
-			(type default)
-		)
-	)
-	(wire
-		(pts
 			(xy 109.22 67.31) (xy 111.76 67.31)
 		)
@@
 		(pts
 			(xy 91.44 67.31) (xy 93.98 67.31)
+		)
+		(stroke
+			(width 0)
+			(type default)
+		)
+	)
+	(wire
+		(pts
+			(xy 104.14 67.31) (xy 109.22 67.31)
 		)
 		(stroke
@@
 	(symbol
 		(lib_id "Device:D_Schottky")
-		(at 101.6 67.31 180)
+		(at 100.33 67.31 180)
 		(unit 1)
 		(exclude_from_sim no)
@@
 		(dnp no)
 		(property "Reference" "D1"
-			(at 101.6 62.484 0)
+			(at 100.33 62.484 0)
 			(effects
 				(font
@@
 		)
 		(property "Value" "SR5200"
-			(at 101.6 64.516 0)
+			(at 100.33 64.516 0)
 			(effects
 				(font
@@
 		)
 		(property "Footprint" "Diode_THT:D_A-405_P7.62mm_Horizontal"
-			(at 101.6 67.31 0)
+			(at 100.33 67.31 0)
 			(effects
 				(font
@@
 		)
 		(property "Datasheet" "https://mm.digikey.com/Volume0/opasdata/d220001/medias/docus/827/SR502-506.pdf"
-			(at 101.6 67.31 0)
+			(at 100.33 67.31 0)
 			(effects
 				(font
@@
 		)
 		(property "Description" "Diodo Schottky"
-			(at 101.6 67.31 0)
+			(at 100.33 67.31 0)
 			(effects
 				(font
@@
 		)
 		(property "Sim.Device" "D"
-			(at 101.6 67.31 0)
+			(at 100.33 67.31 0)
 			(effects
 				(font
@@
 		)
 		(property "Sim.Pins" "1=A 2=K"
-			(at 101.6 67.31 0)
+			(at 100.33 67.31 0)
 			(effects
 				(font
@@
 			)
 		)
-		(property "Value" "22u"
+		(property "Value" "10u"
 			(at 109.474 82.804 0)
 			(effects
@@
 			)
 		)
-		(property "Footprint" "Capacitor_THT:C_Radial_D8.0mm_H11.5mm_P3.50mm"
+		(property "Footprint" "Capacitor_THT:C_Radial_D6.3mm_H7.0mm_P2.50mm"
 			(at 109.22 80.01 0)
 			(effects
@@
 			)
 		)
-		(property "Value" "3m"
+		(property "Value" "2m"
 			(at 90.932 86.106 90)
 			(effects
@@
 			)
 		)
-		(property "Value" "3m"
+		(property "Value" "2m"
 			(at 73.66 65.278 0)
 			(effects

Commit message: PCB prototipo mejorado
Parts:
- removed JP1: Solder Jumper, Jumper:SolderJumper-3_P1.3mm_Open_RoundedPad1.0x1.5mm, symbol Jumper:SolderJumper_3_Open
- removed TP1: Shunt, Resistor_THT:R_Axial_DIN0411_L9.9mm_D3.6mm_P12.70mm_Horizontal, symbol Connector:TestPoint_2Pole
- J2: symbol Connector:Barrel_Jack -> Connector:Barrel_Jack_MountingPin
- J3: footprint Connector_PinHeader_2.54mm:PinHeader_1x02_P2.54mm_Horizontal -> Connector_PinHeader_2.54mm:PinHeader_1x02_P2.54mm_Vertical
- R2: footprint Resistor_THT:R_Axial_DIN0309_L9.0mm_D3.2mm_P2.54mm_Vertical -> Resistor_THT:R_Axial_DIN0309_L9.0mm_D3.2mm_P12.70mm_Horizontal
- TP1: renamed from TP2; footprint Resistor_THT:R_Axial_DIN0411_L9.9mm_D3.6mm_P12.70mm_Horizontal -> Resistor_THT:R_Axial_DIN0411_L9.9mm_D3.6mm_P25.40mm_Horizontal
- TP2: renamed from TP3; footprint Resistor_THT:R_Axial_DIN0411_L9.9mm_D3.6mm_P12.70mm_Horizontal -> Resistor_THT:R_Axial_DIN0411_L9.9mm_D3.6mm_P25.40mm_Horizontal
Connections:
- net +24V: now also L1.2
- net GND: now also TP1.2, TP2.2; no longer L1.4, Q1.3 (S)
- net VCC: now also J1.2 (Pin_2)
- net at C2.2, D1.2 (A): now also L1.4; no longer TP2.1
- net at L1.3: now also TP2.1; no longer TP2.2
- net at C2.1, L1.1: now also Q1.2 (D); no longer TP1.1
- new net: Q1.3 (S), TP1.1
- no-connect marks 0 -> 1
Other:
- moved on the sheet: L1B, Q1, TP1, TP2
