File: epicSEPIC/control.kicad_sch (KiCad schematic)
At the start: 10 parts, among them J4 ICSP, U1 PIC18F4550-IML, U2 1EDN7550U, Y1 20M

Commit message: Agregar datasheets
Parts:
- C4, C5: Part Number (none) -> C0402C200M1RACTU
- R1, R2: Part Number (none) -> ESR03EZPD5102
- R3, R4: value R -> 2; Part Number (none) -> RT0402BRE072RL
- U1: Part Number (none) -> PIC18F4550-IML
- U2: Part Number (none) -> 1EDN7550U
- Y1: Part Number (none) -> FH2000021
Changed lines of the file:
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@@
 			)
 		)
-		(property "Datasheet" "~"
+		(property "Datasheet" "https://www.rohm.com/datasheet?p=ESR03EZPD&dist=Mouser&media=referral&source=mouser.com&campaign=Mouser"
 			(at 152.4 35.56 0)
 			(effects
@@
 		)
 		(property "Description" "Resistor"
+			(at 152.4 35.56 0)
+			(effects
+				(font
+					(size 1.27 1.27)
+				)
+				(hide yes)
+			)
+		)
+		(property "Part Number" "ESR03EZPD5102"
 			(at 152.4 35.56 0)
 			(effects
@@
 		)
 		(property "Description" "Single-Channel EiceDRIVER With True Differential Inputs, 4V UVLO, +4/-8A, SOT-23-6"
+			(at 168.91 38.1 0)
+			(effects
+				(font
+					(size 1.27 1.27)
+				)
+				(hide yes)
+			)
+		)
+		(property "Part Number" "1EDN7550U"
 			(at 168.91 38.1 0)
 			(effects
@@
 			)
 		)
-		(property "Datasheet" "~"
+		(property "Datasheet" "https://www.rohm.com/datasheet?p=ESR03EZPD&dist=Mouser&media=referral&source=mouser.com&campaign=Mouser"
 			(at 152.4 40.64 0)
 			(effects
@@
 		)
 		(property "Description" "Resistor"
+			(at 152.4 40.64 0)
+			(effects
+				(font
+					(size 1.27 1.27)
+				)
+				(hide yes)
+			)
+		)
+		(property "Part Number" "ESR03EZPD5102"
 			(at 152.4 40.64 0)
 			(effects
@@
 			)
 		)
-		(property "Datasheet" "~"
+		(property "Datasheet" "https://content.kemet.com/datasheets/KEM_C1002_X7R_SMD.pdf"
 			(at 24.13 63.5 0)
 			(effects
@@
 		)
 		(property "Description" "Unpolarized capacitor"
+			(at 24.13 63.5 0)
+			(effects
+				(font
+					(size 1.27 1.27)
+				)
+				(hide yes)
+			)
+		)
+		(property "Part Number" "C0402C200M1RACTU"
 			(at 24.13 63.5 0)
 			(effects
@@
 			)
 		)
+		(property "Part Number" "PIC18F4550-IML"
+			(at 88.9 58.42 0)
+			(effects
+				(font
+					(size 1.27 1.27)
+				)
+				(hide yes)
+			)
+		)
 		(pin "18"
 		)
@@
 			)
 		)
-		(property "Value" "R"
+		(property "Value" "2"
 			(at 188.722 34.544 90)
 			(effects
@@
 			)
 		)
-		(property "Datasheet" "~"
+		(property "Datasheet" "https://www.mouser.cl/datasheet/2/447/PYu-RT_1-to-0.01_RoHS_L_9-1222720.pdf"
 			(at 185.42 35.56 0)
 			(effects
@@
 		)
 		(property "Description" "Resistor"
+			(at 185.42 35.56 0)
+			(effects
+				(font
+					(size 1.27 1.27)
+				)
+				(hide yes)
+			)
+		)
+		(property "Part Number" "RT0402BRE072RL"
 			(at 185.42 35.56 0)
 			(effects
@@
 			)
 		)
-		(property "Value" "R"
+		(property "Value" "2"
 			(at 188.722 39.624 90)
 			(effects
@@
 			)
 		)
-		(property "Datasheet" "~"
+		(property "Datasheet" "https://www.mouser.cl/datasheet/2/447/PYu-RT_1-to-0.01_RoHS_L_9-1222720.pdf"
 			(at 185.42 40.64 0)
 			(effects
@@
 			)
 		)
+		(property "Part Number" "RT0402BRE072RL"
+			(at 185.42 40.64 0)
+			(effects
+				(font
+					(size 1.27 1.27)
+				)
+				(hide yes)
+			)
+		)
 		(pin "2"
 		)
@@
 			)
 		)
-		(property "Datasheet" "~"
+		(property "Datasheet" "https://content.kemet.com/datasheets/KEM_C1002_X7R_SMD.pdf"
 			(at 41.91 63.5 0)
 			(effects
@@
 		)
 		(property "Description" "Unpolarized capacitor"
+			(at 41.91 63.5 0)
+			(effects
+				(font
+					(size 1.27 1.27)
+				)
+				(hide yes)
+			)
+		)
+		(property "Part Number" "C0402C200M1RACTU"
 			(at 41.91 63.5 0)
 			(effects
@@
 			)
 		)
-		(property "Datasheet" "~"
+		(property "Datasheet" "https://4donline.ihs.com/images/VipMasterIC/IC/DIOD/DIOD-S-A0003381139/DIOD-S-A0003381139-1.pdf?hkey=CECEF36DEECDED6468708AAF2E19C0C6"
 			(at 33.02 57.15 0)
 			(effects
@@
 			(at 33.02 57.15 0)
 			(effects
+				(font
+					(size 1.27 1.27)
+				)
+				(hide yes)
+			)
+		)
+		(property "Part Number" "FH2000021"
+			(at 33.02 57.15 0)
+			(effects
