File: epicSEPIC/control.kicad_sch (KiCad schematic)
At the start: 10 parts, among them J4 ICSP, U1 PIC18F4550-IML, U2 1EDN7550U, Y1 20M

Commit message: Actualizar BOM
Parts:
- C4, C5: Dist (none) -> Mouser; DistPN (none) -> 80-C0402C200M8HACTU; Mfg (none) -> Kemet; MfgPN (none) -> C0402C200M8HACTU; Part Number C0402C200M1RACTU -> (none)
- R1, R2: Dist (none) -> Mouser; DistPN (none) -> 755-ESR03EZPD5102; Mfg (none) -> Rohm; MfgPN (none) -> ESR03EZPD5102; Part Number ESR03EZPD5102 -> (none)
- R3, R4: Dist (none) -> Mouser; DistPN (none) -> 603-RT0402BRE072RL; Mfg (none) -> Yageo; MfgPN (none) -> RT0402BRE072RL; Part Number RT0402BRE072RL -> (none)
- U1: Dist (none) -> Mouser; DistPN (none) -> 579-PIC18F4550-I/ML; Mfg (none) -> Microchip; MfgPN (none) -> PIC18F4550-IML; Part Number PIC18F4550-IML -> (none)
- U2: Dist (none) -> Mouser; DistPN (none) -> 726-1EDN7550UXTSA1; Mfg (none) -> Infineon; MfgPN (none) -> 1EDN7550U; Part Number 1EDN7550U -> (none)
- Y1: Dist (none) -> Mouser; DistPN (none) -> 729-FH2000021; Mfg (none) -> Diodes Incorporated; MfgPN (none) -> FH2000021; Part Number FH2000021 -> (none)
