File: epicSEPIC/potencia.kicad_sch (KiCad schematic)
At the start: 6 parts, among them Q1 ISZ230N10NM6

Commit message: Agregar datasheets
Parts:
- D1: value D_Schottky -> SK52; Part Number (none) -> SK52
- L1: Part Number (none) -> SRF1280-680M
- Q1: Part Number (none) -> ISZ230N10NM6
Changed lines of the file:
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@@
+			)
+		)
+		(property "Part Number" "SRF1280-680M"
+			(at 165.1 99.06 0)
+			(effects
+				(font
+					(size 1.27 1.27)
+				)
+				(hide yes)
 			)
 		)
@@
 			)
 		)
+		(property "Part Number" "ISZ230N10NM6"
+			(at 142.24 99.06 0)
+			(effects
+				(font
+					(size 1.27 1.27)
+				)
+				(hide yes)
+			)
+		)
 		(pin "1"
 		)
@@
 			)
 		)
-		(property "Datasheet" "~"
+		(property "Datasheet" "https://content.kemet.com/datasheets/KEM_C1002_X7R_SMD.pdf"
 			(at 154.94 88.9 0)
 			(effects
@@
 			)
 		)
-		(property "Value" "D_Schottky"
+		(property "Value" "SK52"
 			(at 171.7675 85.09 0)
 			(effects
@@
 			)
 		)
-		(property "Datasheet" "~"
+		(property "Datasheet" "https://diotec.com/request/datasheet/sk52.pdf"
 			(at 171.45 88.9 0)
 			(effects
@@
 		)
 		(property "Description" "Schottky diode"
+			(at 171.45 88.9 0)
+			(effects
+				(font
+					(size 1.27 1.27)
+				)
+				(hide yes)
+			)
+		)
+		(property "Part Number" "SK52"
 			(at 171.45 88.9 0)
 			(effects
@@
 			(at 130.81 88.9 0)
 			(effects
+				(font
+					(size 1.27 1.27)
+				)
+				(hide yes)
+			)
+		)
+		(property "Part Number" "SRF1280-680M"
+			(at 130.81 88.9 0)
+			(effects

Commit message: Actualizar BOM
Parts:
- C1: Dist (none) -> Mouser; DistPN (none) -> 80-A767KN226M1HLAE50; Mfg (none) -> Kemet; MfgPN (none) -> A767KN226M1HLAE050; Part Number A767KN226M1HLAE050 -> (none)
- C2: Dist (none) -> Mouser; DistPN (none) -> 80-C1206C684M1R; Mfg (none) -> Kemet; MfgPN (none) -> C1206C684M1RACTU; Part Number C1206C684M1RACTU -> (none)
- C3: Dist (none) -> Mouser; DistPN (none) -> 80-A767MU107M1JLAE28; Mfg (none) -> Kemet; MfgPN (none) -> A767MU107M1JLAE28; Part Number A767MU107M1JLAE028 -> (none)
- D1: Dist (none) -> Mouser; DistPN (none) -> 637-SK58; Mfg (none) -> Diotec; MfgPN (none) -> SK58; Part Number SK52 -> (none)
- L1: Dist (none) -> Mouser; DistPN (none) -> 652-SRF1280-680M; Mfg (none) -> Bourns; MfgPN (none) -> SRF1280-680M; Part Number SRF1280-680M -> (none)
- Q1: Dist (none) -> Mouser; DistPN (none) -> 726-ISZ230N10NM6ATMA; Mfg (none) -> Infineon; MfgPN (none) -> ISZ230N10NM6ATMA1; Part Number ISZ230N10NM6 -> (none)
Changed lines of the file:
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@@
 			)
 		)
-		(property "Description" "Polarized capacitor 63Vdc"
+		(property "Description" "Condensador de polímero, 63V"
 			(at 177.8 99.06 0)
 			(effects
@@
 			)
 		)
-		(property "Part Number" "A767MU107M1JLAE028"
+		(property "Dist" "Mouser"
+			(at 177.8 99.06 0)
+			(effects
+				(font
+					(size 1.27 1.27)
+				)
+				(hide yes)
+			)
+		)
+		(property "DistPN" "80-A767MU107M1JLAE28"
+			(at 177.8 99.06 0)
+			(effects
+				(font
+					(size 1.27 1.27)
+				)
+				(hide yes)
+			)
+		)
+		(property "Mfg" "Kemet"
+			(at 177.8 99.06 0)
+			(effects
+				(font
+					(size 1.27 1.27)
+				)
+				(hide yes)
+			)
+		)
+		(property "MfgPN" "A767MU107M1JLAE28"
 			(at 177.8 99.06 0)
 			(effects
@@
 			)
 		)
-		(property "Part Number" "SRF1280-680M"
-			(at 165.1 99.06 0)
+		(property "Dist" "Mouser"
+			(at 165.1 99.06 90)
+			(effects
+				(font
+					(size 1.27 1.27)
+				)
+				(hide yes)
+			)
+		)
+		(property "DistPN" "652-SRF1280-680M"
+			(at 165.1 99.06 90)
+			(effects
+				(font
+					(size 1.27 1.27)
+				)
+				(hide yes)
+			)
+		)
+		(property "Mfg" "Bourns"
+			(at 165.1 99.06 90)
+			(effects
+				(font
+					(size 1.27 1.27)
+				)
+				(hide yes)
+			)
+		)
+		(property "MfgPN" "SRF1280-680M"
+			(at 165.1 99.06 90)
 			(effects
 				(font
@@
 			)
 		)
-		(property "Part Number" "ISZ230N10NM6"
+		(property "Dist" "Mouser"
+			(at 142.24 99.06 0)
+			(effects
+				(font
+					(size 1.27 1.27)
+				)
+				(hide yes)
+			)
+		)
+		(property "DistPN" "726-ISZ230N10NM6ATMA"
+			(at 142.24 99.06 0)
+			(effects
+				(font
+					(size 1.27 1.27)
+				)
+				(hide yes)
+			)
+		)
+		(property "Mfg" "Infineon"
+			(at 142.24 99.06 0)
+			(effects
+				(font
+					(size 1.27 1.27)
+				)
+				(hide yes)
+			)
+		)
+		(property "MfgPN" "ISZ230N10NM6ATMA1"
 			(at 142.24 99.06 0)
 			(effects
@@
 			)
 		)
-		(property "Description" "Unpolarized capacitor 100Vdc"
+		(property "Description" "Condensador cerámico. 100V"
 			(at 154.94 88.9 0)
 			(effects
@@
 			)
 		)
-		(property "Part Number" "C1206C684M1RACTU"
+		(property "Dist" "Mouser"
+			(at 154.94 88.9 90)
+			(effects
+				(font
+					(size 1.27 1.27)
+				)
+				(hide yes)
+			)
+		)
+		(property "DistPN" "80-C1206C684M1R"
+			(at 154.94 88.9 90)
+			(effects
+				(font
+					(size 1.27 1.27)
+				)
+				(hide yes)
+			)
+		)
+		(property "Mfg" "Kemet"
+			(at 154.94 88.9 90)
+			(effects
+				(font
+					(size 1.27 1.27)
+				)
+				(hide yes)
+			)
+		)
+		(property "MfgPN" "C1206C684M1RACTU"
 			(at 154.94 88.9 90)
 			(effects
@@
 			)
 		)
-		(property "Part Number" "SK52"
+		(property "Dist" "Mouser"
+			(at 171.45 88.9 0)
+			(effects
+				(font
+					(size 1.27 1.27)
+				)
+				(hide yes)
+			)
+		)
+		(property "DistPN" "637-SK58"
+			(at 171.45 88.9 0)
+			(effects
+				(font
+					(size 1.27 1.27)
+				)
+				(hide yes)
+			)
+		)
+		(property "Mfg" "Diotec"
+			(at 171.45 88.9 0)
+			(effects
+				(font
+					(size 1.27 1.27)
+				)
+				(hide yes)
+			)
+		)
+		(property "MfgPN" "SK58"
 			(at 171.45 88.9 0)
 			(effects
@@
 			)
 		)
-		(property "Description" "Polarized capacitor 50Vdc"
+		(property "Description" "Condensador de polímero, 50V"
 			(at 118.11 99.06 0)
 			(effects
@@
 			)
 		)
-		(property "Part Number" "A767KN226M1HLAE050"
+		(property "Dist" "Mouser"
+			(at 118.11 99.06 0)
+			(effects
+				(font
+					(size 1.27 1.27)
+				)
+				(hide yes)
+			)
+		)
+		(property "DistPN" "80-A767KN226M1HLAE50"
+			(at 118.11 99.06 0)
+			(effects
+				(font
+					(size 1.27 1.27)
+				)
+				(hide yes)
+			)
+		)
+		(property "Mfg" "Kemet"
+			(at 118.11 99.06 0)
+			(effects
+				(font
+					(size 1.27 1.27)
+				)
+				(hide yes)
+			)
+		)
+		(property "MfgPN" "A767KN226M1HLAE050"
 			(at 118.11 99.06 0)
 			(effects
@@
 			)
 		)
-		(property "Part Number" "SRF1280-680M"
+		(property "Dist" "Mouser"
 			(at 130.81 88.9 0)
 			(effects
+				(font
+					(size 1.27 1.27)
+				)
+				(hide yes)
+			)
+		)
+		(property "DistPN" "652-SRF1280-680M"
+			(at 130.81 88.9 0)
+			(effects
+				(font
+					(size 1.27 1.27)
+				)
+				(hide yes)
+			)
+		)
+		(property "Mfg" "Bourns"
+			(at 130.81 88.9 0)
+			(effects
+				(font
+					(size 1.27 1.27)
+				)
+				(hide yes)
+			)
+		)
+		(property "MfgPN" "SRF1280-680M"
+			(at 130.81 88.9 0)
+			(effects

Commit message: Agregar ESP32 a pcb
Parts:
- D1: value SK52 -> SK58
Changed lines of the file:
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@@
 			)
 		)
-		(property "Description" "Dual Winding Shielded Power Inductor"
+		(property "Description" "Inductor acoplado"
 			(at 165.1 99.06 0)
 			(effects
@@
 			)
 		)
-		(property "Description" "31A Id, 100V Vds, 23mOhm Rds, N-Channel MOSFET, PQFN"
+		(property "Description" "MOSFET Canal N, 31A Id, 100V Vds, 23mOhm Rds"
 			(at 142.24 99.06 0)
 			(effects
@@
 			)
 		)
-		(property "Value" "SK52"
+		(property "Value" "SK58"
 			(at 171.7675 85.09 0)
 			(effects
@@
 			)
 		)
-		(property "Description" "Schottky diode"
+		(property "Description" "Diodo Schottky, 5A, 80V"
 			(at 171.45 88.9 0)
 			(effects
@@
 			)
 		)
-		(property "Description" "Dual Winding Shielded Power Inductor"
+		(property "Description" "Inductor acoplado"
 			(at 130.81 88.9 0)
 			(effects
