File: epicSEPIC/epicSEPIC.kicad_pcb (KiCad board)
At the start: 2 copper layers, 46.6 x 80.3 mm, 52 parts, among them J1 Entrada 24V, J2 USB Tipo B, J3 Salida 12-48V, J4 ICSP, Q1 ISZ230N10NM6, SW1 EN, U1 PIC18F4550-IML, U2 1EDN7550U, U3 TPS54308, U4 TPS54308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

Commit message: ESP32 agregado
Parts:
- RV1: footprint Potentiometer_SMD:Potentiometer_Bourns_3224W_Vertical -> footprints:3313J1102E
- moved R9 2.80 mm to (133.2, 109.2), turned to 180 degrees
- moved RV1 0.57 mm to (131.3, 105.5), turned to 180 degrees
Routing:
- net /Control/PWM: track 1.56 -> 26.1 mm
- net /Monitoreo/Salida: track 17.9 -> 21.7 mm
- net unconnected-(U5-IO4-Pad26): track 2.59 -> 0.00 mm
- net Net-(R9-Pad2): track 1.86 -> 3.66 mm
Other:
- board text added: "Adj"
