File: epicSEPIC/monitoreo.kicad_sch (KiCad schematic)
At the start: 7 parts, among them SW1 EN, U5 ESP32-WROOM-32UE

Commit message: ESP32 agregado
Parts:
- RV1: footprint Potentiometer_SMD:Potentiometer_Bourns_3224W_Vertical -> footprints:3313J1102E
Changed lines of the file:
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@@
 			)
 		)
-		(property "Footprint" "Potentiometer_SMD:Potentiometer_Bourns_3224W_Vertical"
+		(property "Footprint" "footprints:3313J1102E"
 			(at 152.4 124.46 0)
 			(effects
